File: Glavna_ploca_v3.kicad_pcb (KiCad board)
At the start: 2 copper layers, 160 x 110 mm, 85 parts, among them J1 PUMPA1, J10 Granicni prekidac gl, J11 Granicni prekidac gd, J12 Senzor dp, J13 Senzor dz, J14 Senzor gzl, J15 Senzor gzd, J16 Senzor gnl, J17 Senzor gnd, J18 Prekidac za boje, J19 Prekidac za strategije, J2 PUMPA ZA DASKE, J20 Enkoder levi, J21 Enkoder desni, J22 Cinc, J23 Servo, J24 LCD, J25 12V, J26 5V, J27 TMC2209_1, J28 TMC2209_2, J3 PUMPA2, J4 PUMPA3, J5 PUMPA4, J6 Granicni prekidac id, J7 Granicni prekidac il, J8 Granicni prekidac dl, J9 Granicni prekidac dd, Q1 IRLZ44N, Q2 IRLZ44N, Q3 IRLZ44N, Q4 IRLZ44N, Q5 IRLZ44N, U1 NUCLEO-F401RE, U2 TMC2209, U3 TMC2209

Commit message: pcb sa napajanjem
Parts:
- moved J25 319.3 mm to (297.5, 191.0), turned to 90 degrees
- moved J10 293.5 mm to (303.5, 142.5), turned to 90 degrees
- moved R19 286.8 mm to (298.5, 142.0), turned to -90 degrees
- moved R20 284.3 mm to (298.5, 138.0), turned to -90 degrees
- moved J11 278.2 mm to (303.5, 128.5), turned to 90 degrees
- moved R21 271.3 mm to (298.5, 128.0), turned to -90 degrees
- moved R22 269.2 mm to (298.5, 124.0), turned to -90 degrees
- moved J22 254.1 mm to (253.0, 181.0)
- moved J23 251.3 mm to (253.0, 190.0)
- moved R40 208.4 mm to (257.5, 177.0), turned to 180 degrees
- moved R39 206.6 mm to (253.5, 177.0), turned to 180 degrees
- moved R41 189.7 mm to (258.0, 138.5)
- moved R42 189.6 mm to (258.0, 141.0)
- moved R43 181.2 mm to (258.0, 116.5)
- moved R44 179.5 mm to (258.0, 119.0)
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Routing:
- net +5V: track 0.00 -> 354.2 mm
- net +12V: track 0.00 -> 218.5 mm
- added copper zone on F.Cu, net +12V
- added copper zone on F.Cu, net +5V
- added copper zone on B.Cu, net GND
Other:
- board size 160 x 110 mm -> 180 x 117.5 mm
