File: Glavna_ploca_v5.kicad_sch (KiCad schematic)
At the start: 85 parts, among them J1 PUMPA1, J10 Granicni prekidac gl, J11 Granicni prekidac gd, J12 Senzor dp, J13 Senzor dz, J14 Senzor gzl, J15 Senzor gzd, J16 Senzor gnl, J17 Senzor gnd, J18 Prekidac za boje, J19 Prekidac za strategije, J2 PUMPA ZA DASKE, J20 Enkoder levi, J21 Enkoder desni, J22 Cinc, J23 Servo, J24 LCD, J25 12V, J26 5V, J27 TMC2209_1, J28 TMC2209_2, J3 PUMPA2, J4 PUMPA3, J5 PUMPA4, J6 Granicni prekidac id, J7 Granicni prekidac il, J8 Granicni prekidac dl, J9 Granicni prekidac dd, Q1 IRLZ44N, Q2 IRLZ44N, Q3 IRLZ44N, Q4 IRLZ44N, Q5 IRLZ44N, U1 NUCLEO-F401RE, U2 TMC2209, U3 TMC2209

Commit message: konacna ploca
Other:
- moved on the sheet: J28
Changed lines of the file:
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@@
 	(wire
 		(pts
-			(xy 293.37 140.97) (xy 307.34 140.97)
+			(xy 293.37 140.97) (xy 318.77 140.97)
 		)
 		(stroke
@@
 	(wire
 		(pts
-			(xy 297.18 138.43) (xy 307.34 138.43)
+			(xy 297.18 138.43) (xy 318.77 138.43)
 		)
 		(stroke
@@
 	(wire
 		(pts
-			(xy 299.72 135.89) (xy 307.34 135.89)
+			(xy 299.72 135.89) (xy 318.77 135.89)
 		)
 		(stroke
@@
 	(wire
 		(pts
-			(xy 295.91 134.62) (xy 307.34 134.62)
+			(xy 295.91 134.62) (xy 318.77 134.62)
 		)
 		(stroke
@@
 	(wire
 		(pts
-			(xy 307.34 134.62) (xy 307.34 133.35)
+			(xy 318.77 134.62) (xy 318.77 133.35)
 		)
 		(stroke
@@
 	(symbol
 		(lib_id "Connector_Generic:Conn_01x04")
-		(at 312.42 135.89 0)
+		(at 323.85 135.89 0)
 		(unit 1)
 		(exclude_from_sim no)
@@
 		(fields_autoplaced yes)
 		(property "Reference" "J28"
-			(at 314.96 135.8899 0)
+			(at 326.39 135.8899 0)
 			(effects
 				(font
@@
 		)
 		(property "Value" "TMC2209_2"
-			(at 314.96 138.4299 0)
+			(at 326.39 138.4299 0)
 			(effects
 				(font
@@
 		)
 		(property "Footprint" "Connector_JST:JST_XH_B4B-XH-A_1x04_P2.50mm_Vertical"
-			(at 312.42 135.89 0)
+			(at 323.85 135.89 0)
 			(effects
 				(font
@@
 		)
 		(property "Datasheet" "~"
-			(at 312.42 135.89 0)
+			(at 323.85 135.89 0)
 			(effects
 				(font
@@
 		)
 		(property "Description" "Generic connector, single row, 01x04, script generated (kicad-library-utils/schlib/autogen/connector/)"
-			(at 312.42 135.89 0)
+			(at 323.85 135.89 0)
 			(effects
 				(font

Commit message: dodate rupe
Parts:
- added J29: E5V, Connector_JST:JST_XH_B2B-XH-A_1x02_P2.50mm_Vertical, symbol Connector_Generic:Conn_01x02
Connections:
- net +5V: now also J29.1 (Pin_1)
- net at U1.CN7_6 (E5V): now also J29.2 (Pin_2)
- no-connect marks 44 -> 43
Changed lines of the file:
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@@
 	)
 	(no_connect
-		(at 114.3 152.4)
-	)
-	(no_connect
 		(at 109.22 72.39)
 	)
@@
 	(wire
 		(pts
+			(xy 114.3 152.4) (xy 125.73 152.4)
+		)
+		(stroke
+			(width 0)
+			(type default)
+		)
+	)
+	(wire
+		(pts
 			(xy 91.44 363.22) (xy 91.44 365.76)
 		)
@@
 	)
 	(symbol
+		(lib_id "power:+5V")
+		(at 125.73 149.86 0)
+		(unit 1)
+		(exclude_from_sim no)
+		(in_bom yes)
+		(on_board yes)
+		(dnp no)
+		(fields_autoplaced yes)
+		(property "Reference" "#PWR075"
+			(at 125.73 153.67 0)
+			(effects
+				(font
+					(size 1.27 1.27)
+				)
+				(hide yes)
+			)
+		)
+		(property "Value" "+5V"
+			(at 125.73 144.78 0)
+			(effects
+				(font
+					(size 1.27 1.27)
+				)
+			)
+		)
+		(property "Footprint" ""
+			(at 125.73 149.86 0)
+			(effects
+				(font
+					(size 1.27 1.27)
+				)
+				(hide yes)
+			)
+		)
+		(property "Datasheet" ""
+			(at 125.73 149.86 0)
+			(effects
+				(font
+					(size 1.27 1.27)
+				)
+				(hide yes)
+			)
+		)
+		(property "Description" "Power symbol creates a global label with name \"+5V\""
+			(at 125.73 149.86 0)
+			(effects
+				(font
+					(size 1.27 1.27)
+				)
+				(hide yes)
+			)
+		)
+		(pin "1"
+		)
+		(instances
+			(project "Glavna_ploca_v5"
+				(path "/f4e9383e-5eba-4443-ba97-cda3f70ab7b2"
+					(reference "#PWR075")
+					(unit 1)
+				)
+			)
+		)
+	)
+	(symbol
 		(lib_id "power:GND")
 		(at 116.84 373.38 0)
@@
 					(unit 1)
 				)
+			)
+		)
+	)
+	(symbol
+		(lib_id "Connector_Generic:Conn_01x02")
+		(at 130.81 149.86 0)
+		(unit 1)
+		(exclude_from_sim no)
+		(in_bom yes)
+		(on_board yes)
+		(dnp no)
+		(fields_autoplaced yes)
+		(property "Reference" "J29"
+			(at 133.35 149.8599 0)
+			(effects
+				(font
+					(size 1.27 1.27)
+				)
+				(justify left)
+			)
+		)
+		(property "Value" "E5V"
+			(at 133.35 152.3999 0)
+			(effects
+				(font
+					(size 1.27 1.27)
+				)
+				(justify left)
+			)
+		)
+		(property "Footprint" "Connector_JST:JST_XH_B2B-XH-A_1x02_P2.50mm_Vertical"
+			(at 130.81 149.86 0)
+			(effects
+				(font
+					(size 1.27 1.27)
+				)
+				(hide yes)
+			)
+		)
+		(property "Datasheet" "~"
+			(at 130.81 149.86 0)
+			(effects
+				(font
+					(size 1.27 1.27)
+				)
+				(hide yes)
+			)
+		)
+		(property "Description" "Generic connector, single row, 01x02, script generated (kicad-library-utils/schlib/autogen/connector/)"
+			(at 130.81 149.86 0)
+			(effects
+				(font
+					(size 1.27 1.27)
+				)
+				(hide yes)
+			)
+		)
+		(pin "1"
+		)
+		(pin "2"
+		)
+		(instances
+			(project ""
+				(path "/f4e9383e-5eba-4443-ba97-cda3f70ab7b2"
+					(reference "J29")
+					(unit 1)
+				)

Commit message: konacno
Connections:
- net GND: now also U1.CN7_19 (GND_S1), U1.CN7_20 (GND_S1), U1.CN7_22 (GND_S1), U1.CN7_8 (GND_S1)
- no-connect marks 43 -> 42
Changed lines of the file:
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@@
 	)
 	(no_connect
-		(at 114.3 226.06)
-	)
-	(no_connect
 		(at 73.66 77.47)
 	)
@@
 				)
 			)
+		)
+	)
+	(symbol
+		(lib_id "power:GND")
+		(at 114.3 226.06 0)
+		(unit 1)
+		(exclude_from_sim no)
+		(in_bom yes)
+		(on_board yes)
+		(dnp no)
+		(fields_autoplaced yes)
+		(property "Reference" "#PWR076"
+			(at 114.3 232.41 0)
+			(effects
+				(font
+					(size 1.27 1.27)
+				)
+				(hide yes)
+			)
+		)
+		(property "Value" "GND"
+			(at 114.3 231.14 0)
+			(effects
+				(font
+					(size 1.27 1.27)
+				)
+			)
+		)
+		(property "Footprint" ""
+			(at 114.3 226.06 0)
+			(effects
+				(font
+					(size 1.27 1.27)
+				)
+				(hide yes)
+			)
+		)
+		(property "Datasheet" ""
+			(at 114.3 226.06 0)
+			(effects
+				(font
+					(size 1.27 1.27)
+				)
+				(hide yes)
+			)
+		)
+		(property "Description" "Power symbol creates a global label with name \"GND\" , ground"
+			(at 114.3 226.06 0)
+			(effects
+				(font
+					(size 1.27 1.27)
+				)
+				(hide yes)
+			)
+		)
+		(pin "1"
+		)
+		(instances
+			(project ""
+				(path "/f4e9383e-5eba-4443-ba97-cda3f70ab7b2"
+					(reference "#PWR076")
+					(unit 1)
+				)
+			)
