File: Glavna_ploca_v5.kicad_pcb (KiCad board)
At the start: 2 copper layers, 180 x 117.5 mm, 85 parts, among them J1 PUMPA1, J10 Granicni prekidac gl, J11 Granicni prekidac gd, J12 Senzor dp, J13 Senzor dz, J14 Senzor gzl, J15 Senzor gzd, J16 Senzor gnl, J17 Senzor gnd, J18 Prekidac za boje, J19 Prekidac za strategije, J2 PUMPA ZA DASKE, J20 Enkoder levi, J21 Enkoder desni, J22 Cinc, J23 Servo, J24 LCD, J25 12V, J26 5V, J27 TMC2209_1, J28 TMC2209_2, J3 PUMPA2, J4 PUMPA3, J5 PUMPA4, J6 Granicni prekidac id, J7 Granicni prekidac il, J8 Granicni prekidac dl, J9 Granicni prekidac dd, Q1 IRLZ44N, Q2 IRLZ44N, Q3 IRLZ44N, Q4 IRLZ44N, Q5 IRLZ44N, U1 NUCLEO-F401RE, U2 TMC2209, U3 TMC2209

Commit message: konacna ploca
Parts:
- moved J19 14.0 mm to (146.0, 97.0)
- moved R37 14.0 mm to (145.4, 102.0)
- moved R38 14.0 mm to (141.4, 102.0)
- moved J18 14.0 mm to (160.0, 97.0)
- moved R35 14.0 mm to (159.3, 102.2)
- moved R36 14.0 mm to (155.3, 102.2)
- moved R13 10.5 mm to (176.0, 118.0)
- moved R14 10.5 mm to (176.0, 122.0)
- moved J7 10.5 mm to (171.0, 117.5)
- moved J8 10.5 mm to (171.0, 106.9)
- moved R15 10.5 mm to (176.0, 107.5)
- moved R16 10.5 mm to (176.0, 111.5)
Routing:
- net GND: track 0.00 -> 92.1 mm, vias 0 -> 18
- net /STRAT: track 0.00 -> 90.0 mm, vias 0 -> 1
- net /SDA: track 0.00 -> 89.0 mm
- net /SCL: track 0.00 -> 84.2 mm
- net /DIR: track 0.00 -> 83.0 mm
- net /Boja: track 0.00 -> 82.5 mm, vias 0 -> 1
- net /A desni: track 0.00 -> 75.5 mm, vias 0 -> 2
- net /Pumpa 4: track 0.00 -> 71.7 mm, vias 0 -> 2
- net /TMC EN1: track 0.00 -> 71.2 mm, vias 0 -> 4
- net /Pumpa 3: track 0.00 -> 69.7 mm, vias 0 -> 2
- net /GP gl: track 0.00 -> 67.8 mm, vias 0 -> 1
- net /GP gd: track 0.00 -> 59.8 mm, vias 0 -> 1
- net /Pumpa 1: track 0.00 -> 59.1 mm, vias 0 -> 2
- net /Pumpa 5: track 0.00 -> 55.8 mm, vias 0 -> 2
- net /SICK dp: track 0.00 -> 55.0 mm
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
Commit message: dodati nazivi
Parts:
- added G***: LOGO, ftnlogo:ftnlogonovi, F.Cu at (302.0, 165.0)
- added G***: LOGO, notebotlogo:notebotlogo, F.Cu at (149.5, 139.5)
- moved J25 4.03 mm to (301.0, 189.0)
Routing:
- net +12V: track 219.5 -> 232.1 mm
Other:
- board text added: "12V"
- board text added: "5V"
- board text added: "A2 A1 B1 B2"
- board text added: "Cinc"
- board text added: "Enkoder desni"
- board text added: "Enkoder levi"
- board text added: "GP dd"
- board text added: "GP dl"
- board text added: "GP gd"
- board text added: "GP gl"
- board text added: "GP id"
- board text added: "GP il"
- board text added: "LCD"
- board text added: "PUMPA 1"
- board text added: "PUMPA 2"
- board text added: "PUMPA 3"
- board text added: "PUMPA 4"
- board text added: "PUMPA ZA DASKE"
- board text added: "Prekidac za boje"
- board text added: "Prekidac za strategije"
- board text added: "Senzor dp"
- board text added: "Senzor dz"
- board text added: "Senzor gnd"
- board text added: "Senzor gnl"
- board text added: "Senzor gzd"
- board text added: "Senzor gzl"
- board text added: "Servo"

Commit message: dodate rupe
Parts:
- added J29: E5V, Connector_JST:JST_XH_B2B-XH-A_1x02_P2.50mm_Vertical, F.Cu at (151.0, 117.5)
- added REF**: MountingHole_3.2mm_M3_DIN965, MountingHole:MountingHole_3.2mm_M3_DIN965, F.Cu at (307.0, 88.0)
- added REF**: MountingHole_3.2mm_M3_DIN965, MountingHole:MountingHole_3.2mm_M3_DIN965, F.Cu at (136.0, 88.0)
- added REF**: MountingHole_3.2mm_M3_DIN965, MountingHole:MountingHole_3.2mm_M3_DIN965, F.Cu at (136.0, 197.5)
- added REF**: MountingHole_3.2mm_M3_DIN965, MountingHole:MountingHole_3.2mm_M3_DIN965, F.Cu at (306.0, 197.5)
Connections:
- U1 pad CN7_6: unconnected-(U1A-E5V-PadCN7_6) -> Net-(J29-Pin_2)
Routing:
- net Net-(J29-Pin_2): track 0.00 -> 66.9 mm
- net +5V: track 360.0 -> 370.8 mm
Other:
- board size 180 x 117.5 mm -> 180 x 119 mm
- board text added: "E5V"
- board text added: "NOTEBOT"

Commit message: konacno
Connections:
- U1 pad CN7_19: unconnected-(U1A-GND_S1-PadCN7_19)_3 -> GND
- U1 pad CN7_20: unconnected-(U1A-GND_S1-PadCN7_19) -> GND
- U1 pad CN7_22: unconnected-(U1A-GND_S1-PadCN7_19)_2 -> GND
- U1 pad CN7_8: unconnected-(U1A-GND_S1-PadCN7_19)_1 -> GND
Routing:
- net GND: track 92.1 -> 94.3 mm

Commit message: potpisana
Other:
- board text added: "Autori: Luka Ostojić Milica Tešunović Aleksandar Rakić"
Changed lines of the file:
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@@
+		)
+	)
+	(gr_text "Autori: Luka Ostojić\n       Milica Tešunović\n       Aleksandar Rakić\n"
+		(at 309 114.5 90)
+		(layer "F.SilkS")
+		(effects
+			(font
+				(size 1 1)
+				(thickness 0.1)
+			)
+			(justify left bottom)
 		)
 	)
